Commit message: lab7

File: 07-Robot_Arm_1/catkin_ws/src/robot_description/urdf/husky.urdf.xacro (robot description, xacro)
@@ -101,5 +101,13 @@
     <origin xyz="${wheelbase/2} ${track/2} ${wheel_vertical_offset}" rpy="0 0 0" />
   </xacro:husky_wheel>
-  <!-- TODO -->
+  <xacro:husky_wheel wheel_prefix="back_left">
+    <origin xyz="${-wheelbase/2} ${track/2} ${wheel_vertical_offset}" rpy="0 0 0"/>
+  </xacro:husky_wheel>
+    <xacro:husky_wheel wheel_prefix="back_right">
+    <origin xyz="${-wheelbase/2} ${-track/2} ${wheel_vertical_offset}" rpy="0 0 0"/>
+  </xacro:husky_wheel>
+    <xacro:husky_wheel wheel_prefix="front_right">
+    <origin xyz="${wheelbase/2} ${-track/2} ${wheel_vertical_offset}" rpy="0 0 0"/>
+  </xacro:husky_wheel>
   <xacro:husky_decorate />
   <xacro:if value="$(arg laser_enabled)">
